Commit message: added a new usd. working on fixes to the reset on trajectory. Added more plotting to debug the weird elbow joint

File: robot_assets/g1/g1_21j/g1_21j.urdf (robot description, URDF)
Before this commit: robot g1_21j, 64 links, 63 joints
Links:
- link head_link: geometry visual mesh filename=meshes/head_link.STL
- link left_ankle_pitch_link: geometry visual mesh filename=meshes/left_ankle_pitch_link.STL
- link left_ankle_roll_link: geometry collision sphere radius=0.005; collision sphere radius=0.005
- link left_elbow_link: geometry collision cylinder length=0.22 radius=0.035; visual mesh filename=meshes/left_elbow_link.STL
- link left_hand_index_0_link: geometry visual mesh filename=meshes/left_hand_index_0_link.STL
- link left_hand_index_1_link: geometry visual mesh filename=meshes/left_hand_index_1_link.STL
- link left_hand_middle_0_link: geometry visual mesh filename=meshes/left_hand_middle_0_link.STL
- link left_hand_middle_1_link: geometry visual mesh filename=meshes/left_hand_middle_1_link.STL
- link left_hand_palm_link: geometry visual mesh filename=meshes/left_hand_palm_link.STL
- link left_hand_thumb_0_link: geometry visual mesh filename=meshes/left_hand_thumb_0_link.STL
- link left_hand_thumb_1_link: geometry visual mesh filename=meshes/left_hand_thumb_1_link.STL
- link left_hand_thumb_2_link: geometry visual mesh filename=meshes/left_hand_thumb_2_link.STL
- link left_hip_pitch_link: geometry visual mesh filename=meshes/left_hip_pitch_link.STL
- link left_hip_roll_link: geometry collision cylinder length=0.25 radius=0.045; visual mesh filename=meshes/left_hip_roll_link.STL
- link left_hip_yaw_link: geometry visual mesh filename=meshes/left_hip_yaw_link.STL
- link left_knee_link: geometry collision cylinder length=0.3 radius=0.05; visual mesh filename=meshes/left_knee_link.STL
- link left_shoulder_pitch_link: geometry visual mesh filename=meshes/left_shoulder_pitch_link.STL
- link left_shoulder_roll_link: geometry visual mesh filename=meshes/left_shoulder_roll_link.STL
- link left_shoulder_yaw_link: geometry visual mesh filename=meshes/left_shoulder_yaw_link.STL
- link left_wrist_pitch_link: geometry visual mesh filename=meshes/left_wrist_pitch_link.STL
- link left_wrist_roll_link: geometry visual mesh filename=meshes/left_wrist_roll_link.STL
- link left_wrist_yaw_link: geometry collision sphere radius=0.055; visual mesh filename=meshes/left_wrist_yaw_link.STL
- link logo_link: geometry visual mesh filename=meshes/logo_link.STL
- link pelvis_contour_link: geometry visual mesh filename=meshes/pelvis_contour_link.STL
- link pelvis_link: geometry visual mesh filename=meshes/pelvis.STL
- link right_ankle_pitch_link: geometry visual mesh filename=meshes/right_ankle_pitch_link.STL
- link right_ankle_roll_link: geometry collision sphere radius=0.005; collision sphere radius=0.005
- link right_elbow_link: geometry collision cylinder length=0.22 radius=0.035; visual mesh filename=meshes/right_elbow_link.STL
- link right_hand_index_0_link: geometry visual mesh filename=meshes/right_hand_index_0_link.STL
- link right_hand_index_1_link: geometry visual mesh filename=meshes/right_hand_index_1_link.STL
- link right_hand_middle_0_link: geometry visual mesh filename=meshes/right_hand_middle_0_link.STL
- link right_hand_middle_1_link: geometry visual mesh filename=meshes/right_hand_middle_1_link.STL
- link right_hand_palm_link: geometry visual mesh filename=meshes/right_hand_palm_link.STL
- link right_hand_thumb_0_link: geometry visual mesh filename=meshes/right_hand_thumb_0_link.STL
- link right_hand_thumb_1_link: geometry visual mesh filename=meshes/right_hand_thumb_1_link.STL
- link right_hand_thumb_2_link: geometry visual mesh filename=meshes/right_hand_thumb_2_link.STL
- link right_hip_pitch_link: geometry visual mesh filename=meshes/right_hip_pitch_link.STL
- link right_hip_roll_link: geometry collision cylinder length=0.25 radius=0.045; visual mesh filename=meshes/right_hip_roll_link.STL
- link right_hip_yaw_link: geometry visual mesh filename=meshes/right_hip_yaw_link.STL
- link right_knee_link: geometry collision cylinder length=0.3 radius=0.05; visual mesh filename=meshes/right_knee_link.STL
- link right_shoulder_pitch_link: geometry visual mesh filename=meshes/right_shoulder_pitch_link.STL
- link right_shoulder_roll_link: geometry visual mesh filename=meshes/right_shoulder_roll_link.STL
- link right_shoulder_yaw_link: geometry visual mesh filename=meshes/right_shoulder_yaw_link.STL
- link right_wrist_pitch_link: geometry visual mesh filename=meshes/right_wrist_pitch_link.STL
- link right_wrist_roll_link: geometry visual mesh filename=meshes/right_wrist_roll_link.STL
- link right_wrist_yaw_link: geometry collision sphere radius=0.055; visual mesh filename=meshes/right_wrist_yaw_link.STL
- link torso_link: geometry visual mesh filename=meshes/torso_link.STL
- link waist_roll_link: geometry visual mesh filename=meshes/waist_roll_link.STL
- link waist_support_link: geometry visual mesh filename=meshes/waist_support_link.STL
- link waist_yaw_link: geometry collision box size=0.12 0.175 0.4; visual mesh filename=meshes/waist_yaw_link.STL
